Commit message: Se a;aden variables para construir el robot

File: my_robot_description/urdf/my_robot4.urdf.xacro (robot description, xacro)
@@ -1,4 +1,9 @@
 <?xml version="1.0"?>
 <robot name="my_robot" xmlns:xacro="http://www.ros.org.wiki/xacro">
+    <xacro:property name="base_length" value="0.60" />
+    <xacro:property name="base_width" value="0.40" />
+    <xacro:property name="base_height" value="0.20" />
+    <xacro:property name="wheel_radius" value="0.10" />
+    <xacro:property name="wheel_length" value="0.05" />
     <material name="green">
         <color rgba="0.0 0.5 0.0 1.0"/>
@@ -15,7 +20,7 @@
         <visual>
             <geometry>
-                <box size="0.60 0.40 0.20"/>
+                <box size="${base_length} ${base_width} ${base_height}"/>
             </geometry>
-            <origin xyz="0.0 0.0 0.10" rpy="0.0 0.0 0.0"/>
+            <origin xyz="0.0 0.0 ${base_height/2.0}" rpy="0.0 0.0 0.0"/>
             <material name="blue"/>
         </visual>
@@ -24,7 +29,7 @@
         <visual>
             <geometry>
-                <cylinder radius="0.10" length="0.050"/>
+                <cylinder radius="${wheel_radius}" length="${wheel_length}"/>
             </geometry>
-            <origin xyz="0.0 0.0 0.0" rpy="1.57 0 0"/>
+            <origin xyz="0.0 0.0 0.0" rpy="${pi/2.0} 0 0"/>
             <material name="grey"/>
         </visual>
@@ -33,7 +38,7 @@
         <visual>
             <geometry>
-                <cylinder radius="0.10" length="0.05"/>
+                <cylinder radius="${wheel_radius}" length="${wheel_length}"/>
             </geometry>
-            <origin xyz="0.0 0.0 0.0" rpy="1.57 0.0 0.0"/>
+            <origin xyz="0.0 0.0 0.0" rpy="${pi/2.0} 0.0 0.0"/>
             <material name="grey"/>
         </visual>
@@ -56,5 +61,5 @@
         <parent link="base_link"/>
         <child link="right_wheel_link"/>
-        <origin xyz="-0.15 -0.225 0" rpy="0.0 0.0 0.0"/>
+        <origin xyz="${-base_length/4.0}  ${-(base_width+wheel_length)/2.0} 0" rpy="0.0 0.0 0.0"/>
         <axis xyz="0.0 1.0 0"/>
     </joint>
@@ -62,5 +67,5 @@
         <parent link="base_link"/>
         <child link="left_wheel_link"/>
-        <origin xyz="-0.15 0.225 0" rpy="0.0 0.0 0.0"/>
+        <origin xyz="${-base_length/4.0}  ${(base_width+wheel_length)/2.0} 0" rpy="0.0 0.0 0.0"/>
         <axis xyz="0.0 1.0 0.0"/>
     </joint>
@@ -68,5 +73,5 @@
         <parent link="base_link"/>
         <child link="caster_wheel_link"/>
-        <origin xyz="0.2 0.0 -0.05" rpy="0.0 0.0 0.0"/>
+        <origin xyz="${base_length/3.0} 0.0 -0.05" rpy="0.0 0.0 0.0"/>
         <axis xyz="0.0 1.0 0.0"/>
     </joint>

Commit message: Se a;aden variables para construir el robot 2

File: my_robot_description/urdf/my_robot4.urdf.xacro (robot description, xacro)
@@ -47,5 +47,5 @@
         <visual>
             <geometry>
-                <sphere radius="0.05"/>
+                <sphere radius="${wheel_radius/2}"/>
             </geometry>
             <origin xyz="0.0 0.0 0.0" rpy="0.0 0.0 0.0"/>
@@ -73,5 +73,5 @@
         <parent link="base_link"/>
         <child link="caster_wheel_link"/>
-        <origin xyz="${base_length/3.0} 0.0 -0.05" rpy="0.0 0.0 0.0"/>
+        <origin xyz="${base_length/3.0} 0.0 ${-wheel_radius/2.0}" rpy="0.0 0.0 0.0"/>
         <axis xyz="0.0 1.0 0.0"/>
     </joint>

Commit message: Se a;aden variables para construir el robot 2

File: my_robot_description/urdf/my_robot4.urdf.xacro (robot description, xacro)
@@ -56,5 +56,5 @@
         <parent link="base_footprint"/>
         <child link="base_link"/>
-        <origin xyz="0.0 0.0 0.1" rpy="0.0 0.0 0.0"/>
+        <origin xyz="0.0 0.0 ${wheel_radius}" rpy="0.0 0.0 0.0"/>
     </joint>
     <joint name="base_right_wheel_joint" type="continuous">

Commit message: Example de Xacro Macro funcion

File: my_robot_description/urdf/my_robot4.urdf.xacro (robot description, xacro)
@@ -6,4 +6,14 @@
     <xacro:property name="wheel_radius" value="0.10" />
     <xacro:property name="wheel_length" value="0.05" />
+    <xacro:macro name="example_macro" params="a b c">
+        <link name="dummy_link">
+            <visual>
+                <geometry>
+                    <box size="${a} ${b} ${c}"/>
+                </geometry>
+            </visual>
+        </link>
+    </xacro:macro>
+    <xacro:example_macro a="2" b="4" c="s" />
     <material name="green">
         <color rgba="0.0 0.5 0.0 1.0"/>

Commit message: Se genera xacro macro para las ruenas izq der

File: my_robot_description/urdf/my_robot4.urdf.xacro (robot description, xacro)
@@ -1,19 +1,4 @@
 <?xml version="1.0"?>
 <robot name="my_robot" xmlns:xacro="http://www.ros.org.wiki/xacro">
-    <xacro:property name="base_length" value="0.60" />
-    <xacro:property name="base_width" value="0.40" />
-    <xacro:property name="base_height" value="0.20" />
-    <xacro:property name="wheel_radius" value="0.10" />
-    <xacro:property name="wheel_length" value="0.05" />
-    <xacro:macro name="example_macro" params="a b c">
-        <link name="dummy_link">
-            <visual>
-                <geometry>
-                    <box size="${a} ${b} ${c}"/>
-                </geometry>
-            </visual>
-        </link>
-    </xacro:macro>
-    <xacro:example_macro a="2" b="4" c="s" />
     <material name="green">
         <color rgba="0.0 0.5 0.0 1.0"/>
@@ -25,4 +10,22 @@
         <color rgba="0.5 0.5 0.5 1.0"/>
     </material>
+    <xacro:property name="base_length" value="0.60" />
+    <xacro:property name="base_width" value="0.40" />
+    <xacro:property name="base_height" value="0.20" />
+    <xacro:property name="wheel_radius" value="0.10" />
+    <xacro:property name="wheel_length" value="0.05" />
+    <xacro:macro name="wheel_link" params="prefix">
+        <link name="${prefix}_wheel_link">
+            <visual>
+                <geometry>
+                    <cylinder radius="${wheel_radius}" length="${wheel_length}"/>
+                </geometry>
+                <origin xyz="0.0 0.0 0.0" rpy="${pi/2.0} 0.0 0.0"/>
+                <material name="grey"/>
+            </visual>
+        </link>
+    </xacro:macro>
+    <xacro:wheel_link prefix="left"/>
+    <xacro:wheel_link prefix="right"/>
     <link name="base_footprint">
     </link>
@@ -34,22 +37,4 @@
             <origin xyz="0.0 0.0 ${base_height/2.0}" rpy="0.0 0.0 0.0"/>
             <material name="blue"/>
-        </visual>
-    </link>
-    <link name="right_wheel_link">
-        <visual>
-            <geometry>
-                <cylinder radius="${wheel_radius}" length="${wheel_length}"/>
-            </geometry>
-            <origin xyz="0.0 0.0 0.0" rpy="${pi/2.0} 0 0"/>
-            <material name="grey"/>
-        </visual>
-    </link>
-    <link name="left_wheel_link">
-        <visual>
-            <geometry>
-                <cylinder radius="${wheel_radius}" length="${wheel_length}"/>
-            </geometry>
-            <origin xyz="0.0 0.0 0.0" rpy="${pi/2.0} 0.0 0.0"/>
-            <material name="grey"/>
         </visual>
     </link>

Commit message: Se vuelve al urdf original

File: my_robot_description/urdf/my_robot4.urdf.xacro (robot description, xacro)
@@ -1,4 +1,9 @@
 <?xml version="1.0"?>
 <robot name="my_robot" xmlns:xacro="http://www.ros.org.wiki/xacro">
+    <xacro:property name="base_length" value="0.60" />
+    <xacro:property name="base_width" value="0.40" />
+    <xacro:property name="base_height" value="0.20" />
+    <xacro:property name="wheel_radius" value="0.10" />
+    <xacro:property name="wheel_length" value="0.05" />
     <material name="green">
         <color rgba="0.0 0.5 0.0 1.0"/>
@@ -10,22 +15,4 @@
         <color rgba="0.5 0.5 0.5 1.0"/>
     </material>
-    <xacro:property name="base_length" value="0.60" />
-    <xacro:property name="base_width" value="0.40" />
-    <xacro:property name="base_height" value="0.20" />
-    <xacro:property name="wheel_radius" value="0.10" />
-    <xacro:property name="wheel_length" value="0.05" />
-    <xacro:macro name="wheel_link" params="prefix">
-        <link name="${prefix}_wheel_link">
-            <visual>
-                <geometry>
-                    <cylinder radius="${wheel_radius}" length="${wheel_length}"/>
-                </geometry>
-                <origin xyz="0.0 0.0 0.0" rpy="${pi/2.0} 0.0 0.0"/>
-                <material name="grey"/>
-            </visual>
-        </link>
-    </xacro:macro>
-    <xacro:wheel_link prefix="left"/>
-    <xacro:wheel_link prefix="right"/>
     <link name="base_footprint">
     </link>
@@ -37,4 +24,22 @@
             <origin xyz="0.0 0.0 ${base_height/2.0}" rpy="0.0 0.0 0.0"/>
             <material name="blue"/>
+        </visual>
+    </link>
+    <link name="right_wheel_link">
+        <visual>
+            <geometry>
+                <cylinder radius="${wheel_radius}" length="${wheel_length}"/>
+            </geometry>
+            <origin xyz="0.0 0.0 0.0" rpy="${pi/2.0} 0 0"/>
+            <material name="grey"/>
+        </visual>
+    </link>
+    <link name="left_wheel_link">
+        <visual>
+            <geometry>
+                <cylinder radius="${wheel_radius}" length="${wheel_length}"/>
+            </geometry>
+            <origin xyz="0.0 0.0 0.0" rpy="${pi/2.0} 0.0 0.0"/>
+            <material name="grey"/>
         </visual>
     </link>

Commit message: Se crean archivos individuales para las prpoiedades comunes y el objeto base

File: my_robot_description/urdf/my_robot4.urdf.xacro (robot description, xacro)
@@ -1,4 +1,5 @@
 <?xml version="1.0"?>
 <robot name="my_robot" xmlns:xacro="http://www.ros.org.wiki/xacro">
+    <xacro:include filename="common_properties.xacro"/>
     <xacro:property name="base_length" value="0.60" />
     <xacro:property name="base_width" value="0.40" />
@@ -6,13 +7,4 @@
     <xacro:property name="wheel_radius" value="0.10" />
     <xacro:property name="wheel_length" value="0.05" />
-    <material name="green">
-        <color rgba="0.0 0.5 0.0 1.0"/>
-    </material>
-    <material name="blue">
-        <color rgba="0.0 0.0 0.5 1.0"/>
-    </material>
-    <material name="grey">
-        <color rgba="0.5 0.5 0.5 1.0"/>
-    </material>
     <link name="base_footprint">
     </link>

Commit message: Se imprtan los files .xacro coin propiedades y los valores comunes en archivos separados

File: my_robot_description/urdf/my_robot4.urdf.xacro (robot description, xacro)
@@ -2,69 +2,4 @@
 <robot name="my_robot" xmlns:xacro="http://www.ros.org.wiki/xacro">
     <xacro:include filename="common_properties.xacro"/>
-    <xacro:property name="base_length" value="0.60" />
-    <xacro:property name="base_width" value="0.40" />
-    <xacro:property name="base_height" value="0.20" />
-    <xacro:property name="wheel_radius" value="0.10" />
-    <xacro:property name="wheel_length" value="0.05" />
-    <link name="base_footprint">
-    </link>
-    <link name="base_link">
-        <visual>
-            <geometry>
-                <box size="${base_length} ${base_width} ${base_height}"/>
-            </geometry>
-            <origin xyz="0.0 0.0 ${base_height/2.0}" rpy="0.0 0.0 0.0"/>
-            <material name="blue"/>
-        </visual>
-    </link>
-    <link name="right_wheel_link">
-        <visual>
-            <geometry>
-                <cylinder radius="${wheel_radius}" length="${wheel_length}"/>
-            </geometry>
-            <origin xyz="0.0 0.0 0.0" rpy="${pi/2.0} 0 0"/>
-            <material name="grey"/>
-        </visual>
-    </link>
-    <link name="left_wheel_link">
-        <visual>
-            <geometry>
-                <cylinder radius="${wheel_radius}" length="${wheel_length}"/>
-            </geometry>
-            <origin xyz="0.0 0.0 0.0" rpy="${pi/2.0} 0.0 0.0"/>
-            <material name="grey"/>
-        </visual>
-    </link>
-    <link name="caster_wheel_link">
-        <visual>
-            <geometry>
-                <sphere radius="${wheel_radius/2}"/>
-            </geometry>
-            <origin xyz="0.0 0.0 0.0" rpy="0.0 0.0 0.0"/>
-            <material name="grey"/>
-        </visual>
-    </link>
-    <joint name="base_joint" type="fixed">
-        <parent link="base_footprint"/>
-        <child link="base_link"/>
-        <origin xyz="0.0 0.0 ${wheel_radius}" rpy="0.0 0.0 0.0"/>
-    </joint>
-    <joint name="base_right_wheel_joint" type="continuous">
-        <parent link="base_link"/>
-        <child link="right_wheel_link"/>
-        <origin xyz="${-base_length/4.0}  ${-(base_width+wheel_length)/2.0} 0" rpy="0.0 0.0 0.0"/>
-        <axis xyz="0.0 1.0 0"/>
-    </joint>
-    <joint name="base_left_wheel_joint" type="continuous">
-        <parent link="base_link"/>
-        <child link="left_wheel_link"/>
-        <origin xyz="${-base_length/4.0}  ${(base_width+wheel_length)/2.0} 0" rpy="0.0 0.0 0.0"/>
-        <axis xyz="0.0 1.0 0.0"/>
-    </joint>
-    <joint name="base_caster_wheel_joint" type="fixed">
-        <parent link="base_link"/>
-        <child link="caster_wheel_link"/>
-        <origin xyz="${base_length/3.0} 0.0 ${-wheel_radius/2.0}" rpy="0.0 0.0 0.0"/>
-        <axis xyz="0.0 1.0 0.0"/>
-    </joint>
+     <xacro:include filename="mobile_base.xacro"/>
 </robot>
