Commit message: Se a;ade la matriz de inertia para el base_link con lantilla en common properties

File: my_robot_description/urdf/common_properties.xacro (robot description, xacro)
@@ -10,3 +10,12 @@
         <color rgba="0.5 0.5 0.5 1.0"/>
     </material>
+    <xacro:macro name="box_inertia" params="m x y z o_xyz o_rpy">
+        <inertial>
+            <mass value="${m}"/>
+            <origin xyz="${o_xyz}" rpy="${o_rpy}"/>
+            <inertia ixx="${(m/12) * (y*y + z*z)}" ixy="0"                        ixz="0"
+                                                   iyy="${(m/12) * (x*x + z*z)}"  iyz="0"
+                                                                                  izz="${(m/12) * (y*y + x*x)}" />
+        </inertial>
+    </xacro:macro>
 </robot>

File: my_robot_description/urdf/mobile_base.xacro (robot description, xacro)
@@ -16,4 +16,6 @@
             <material name="blue"/>
         </visual>
+        <xacro:box_inertia m="5.0" x="${base_length}" y="${base_width}" z="${base_height}"
+                            o_xyz="0.0 0.0 ${base_height/2.0}" o_rpy="0.0 0.0 0.0"/>
     </link>
     <link name="right_wheel_link">

Commit message: Se a;ade las inertias a box wheels y spheres

File: my_robot_description/urdf/common_properties.xacro (robot description, xacro)
@@ -19,3 +19,21 @@
         </inertial>
     </xacro:macro>
+    <xacro:macro name="cilinder_inertia" params="m r h o_xyz o_rpy">
+        <inertial>
+            <mass value="${m}"/>
+            <origin xyz="${o_xyz}" rpy="${o_rpy}"/>
+            <inertia ixx="${(m/12) * (3*r*r + h*h)}" ixy="0"                          ixz="0"
+                                                     iyy="${(m/12) * (3*r*r + h*h)}"  iyz="0"
+                                                                                      izz="${(m*r*r)/2}" />
+        </inertial>
+    </xacro:macro>
+    <xacro:macro name="sphere_inertia" params="m r o_xyz o_rpy">
+        <inertial>
+            <mass value="${m}"/>
+            <origin xyz="${o_xyz}" rpy="${o_rpy}"/>
+            <inertia ixx="${(2*m*r*r)/5}"   ixy="0"               ixz="0"
+                                            iyy="${(2*m*r*r)/5}"  iyz="0"
+                                                                  izz="${(2*m*r*r)/5}" />
+        </inertial>
+    </xacro:macro>
 </robot>

File: my_robot_description/urdf/mobile_base.xacro (robot description, xacro)
@@ -27,4 +27,6 @@
             <material name="grey"/>
         </visual>
+        <xacro:cilinder_inertia m="1.0" r="${wheel_radius}" h="${wheel_length}"
+                            o_xyz="0.0 0.0 0.0" o_rpy="${pi/2.0} 0.0 0.0"/>
     </link>
     <link name="left_wheel_link">
@@ -36,4 +38,6 @@
             <material name="grey"/>
         </visual>
+        <xacro:cilinder_inertia m="1.0" r="${wheel_radius}" h="${wheel_length}"
+                            o_xyz="0.0 0.0 0.0" o_rpy="${pi/2.0} 0.0 0.0"/>
     </link>
     <link name="caster_wheel_link">
@@ -45,4 +49,6 @@
             <material name="grey"/>
         </visual>
+        <xacro:sphere_inertia m="0.5" r="${wheel_radius/2}"
+                            o_xyz="0.0 0.0 0.0" o_rpy="0.0 0.0 0.0"/>
     </link>
     <joint name="base_joint" type="fixed">

Commit message: Mi primera version del brazo, junto al robot

File: my_robot_description/urdf/common_properties.xacro (robot description, xacro)
@@ -9,4 +9,10 @@
     <material name="grey">
         <color rgba="0.5 0.5 0.5 1.0"/>
+    </material>
+    <material name="orange">
+        <color rgba="0.90 0.32 0.00 1.0"/>
+    </material>
+    <material name="yellow">
+        <color rgba="1.00 0.76 0.03 1.0"/>
     </material>
     <xacro:macro name="box_inertia" params="m x y z o_xyz o_rpy">

File: my_robot_description/urdf/my_robot4.urdf.xacro (robot description, xacro)
@@ -5,3 +5,9 @@
     <xacro:include filename="mobile_base_gazebo.xacro"/>
     <xacro:include filename="camera.xacro" />
+    <xacro:include filename="standalone_arm.urdf.xacro" />
+    <joint name="robot_to_base" type="fixed">
+        <parent link="base_link"/>
+        <child link="arm_base_link"/>
+        <origin xyz="${base_length/2 - arm_base_width} 0 ${base_height+(arm_base_height/2)}" rpy="0 0 0"/>
+    </joint>
 </robot>
