Commit message: Se añade friccion con dynamics

File: my_robot_description/urdf/arm.xacro (robot description, xacro)
@@ -57,5 +57,5 @@
                             o_xyz="0.0 0.0 0.0" o_rpy="${pi/2.0} 0.0 0.0"/>
     </link>
-    <joint name="base_forearm_joint" type="revolute">
+    <joint name="arm_base_forearm_joint" type="revolute">
         <parent link="arm_base_link"/>
         <child link="forearm_link"/>
@@ -63,6 +63,7 @@
         <axis xyz="0.0 1.0 0"/>
         <limit lower="0" upper="${pi/2}" effort="100.0" velocity="100"/>
+        <dynamics damping="0.3" friction="0.3"/>
     </joint>
-    <joint name="forearm_hand_link_joint" type="revolute">
+    <joint name="forearm_hand_joint" type="revolute">
         <parent link="forearm_link"/>
         <child link="hand_link"/>
@@ -70,4 +71,5 @@
         <axis xyz="0.0 1.0 0.0"/>
         <limit lower="0" upper="${pi/2}" effort="100.0" velocity="100.0"/>
+        <dynamics damping="0.3" friction="0.3"/>
     </joint>
 </robot>

Commit message: Se modifica la carga de archivps en mobile_base se corrige la posicion de las inertcias del braxo

File: my_robot_description/urdf/arm.xacro (robot description, xacro)
@@ -20,5 +20,5 @@
             <origin xyz="0.0 0.0 ${arm_base_height}" rpy="0.0 0.0 0.0"/>
         </collision>
-        <xacro:box_inertia m="5.0" x="${arm_base_length}" y="${arm_base_width}" z="${arm_base_height}"
+        <xacro:box_inertia m="0.5" x="${arm_base_length}" y="${arm_base_width}" z="${arm_base_height}"
                             o_xyz="0.0 0.0 ${arm_base_height/2.0}" o_rpy="0.0 0.0 0.0"/>
     </link>
@@ -38,5 +38,5 @@
         </collision>
         <xacro:cilinder_inertia m="1.0" r="${arm_radius}" h="${arm_length}"
-                            o_xyz="0.0 0.0 0.0" o_rpy="${pi/2.0} 0.0 0.0"/>
+                            o_xyz="0.0 0.0 ${arm_length/2}" o_rpy="0.0 0.0 0.0"/>
     </link>
     <link name="hand_link">
@@ -55,5 +55,5 @@
         </collision>
         <xacro:cilinder_inertia m="1.0" r="${arm_radius}" h="${arm_length}"
-                            o_xyz="0.0 0.0 0.0" o_rpy="${pi/2.0} 0.0 0.0"/>
+                            o_xyz="0.0 0.0 ${arm_length/2}" o_rpy="0.0 0.0 0.0"/>
     </link>
     <joint name="arm_base_forearm_joint" type="revolute">

File: my_robot_description/urdf/my_robot4.urdf.xacro (robot description, xacro)
@@ -5,6 +5,7 @@
     <xacro:include filename="mobile_base_gazebo.xacro"/>
     <xacro:include filename="camera.xacro" />
-    <xacro:include filename="standalone_arm.urdf.xacro" />
-    <joint name="robot_to_base" type="fixed">
+    <xacro:include filename="arm.xacro" />
+    <xacro:include filename="arm_gazebo.xacro" />
+    <joint name="mobile_base_arm_joint" type="fixed">
         <parent link="base_link"/>
         <child link="arm_base_link"/>
